File: kicad/80bus.kicad_pcb (KiCad board)
At the start: 2 copper layers, 203.2 x 203.2 mm, 78 parts, among them J1 Conn_01x80NasBus, Q1 2N3904, SW1 SW_DIP_x06, SW2 SW_SPDT, U1 74LS244, U10 74LS04, U100 2764, U101 2764, U102 2764, U103 2764, U11 74LS00, U12 74LS30, U2 DecodeHeader, U200 MK36000_8K_ROM, U201 2764, U3 74LS244, U4 74159, U5 74LS244, U6 74LS175, U7 74LS32, U8 7406, U9 74LS20

Commit message: Update docs
Parts:
- added G001: LOGO, 80bus:qr-code, B.Cu at (150.7, 227.9)
- moved JP1 0.06 mm to (253.4, 75.9)
Routing:
- net VCC: track 1474.0 -> 1474.6 mm
Other:
- board text added: "CS-002"
- board text added: "Copyright (c) Codesqueak - 2025 - All Rights Reserved"
- board text added: "Docs -->"
- board text added: "Errata 1.2 -> 2.3 - Convert to KiCad 9"
- board text added: "Version 2.3"
- board text added: "b03c65fd-131e-4edc-b2dc-b6777f3aa3c5"
- board text removed: "310f6188-d04e-46a9-8d86-e9c22f007e7a"
- board text removed: "Copyright (c) Codesqueak - 2023 - All Rights Reserved"
- board text removed: "Errata 1.3.0 -> 2.0.0 - Convert to KiCad 7 - Change switch types - Minor track improvements"
- board text removed: "Version 2.0.0"
