File: kicad/80bus.kicad_sch (KiCad schematic)
At the start: 77 parts, among them J1 Conn_01x80NasBus, Q1 2N3904, SW1 SW_DIP_x06, SW2 SW_SPDT, U1 74LS244, U10 74LS04, U100 2764, U101 2764, U102 2764, U103 2764, U11 74LS00, U12 74LS30, U2 DecodeHeader, U200 MK36000_8K_ROM, U201 2764, U3 74LS244, U4 74159, U5 74LS244, U6 74LS175, U7 74LS32, U8 7406, U9 74LS20

Commit message: Update docs
Other:
- moved on the sheet: R16
